File: volume_control_and_pc_busy_simulator/schematic/schematic.kicad_sch (KiCad schematic)
At the start: 8 parts, among them SW1 RotaryEncoder_Switch, SW2 SW_Push, SW3 SW_Push, U1 Sparkfun_Pro_Micro

Commit message: VolumeControl: Schematic update
Parts:
- D1, D2: footprint LED_THT:LED_D5.0mm_Horizontal_O1.27mm_Z15.0mm -> LED_THT:LED_D5.0mm
Connections:
- no-connect marks 0 -> 15
Changed lines of the file:
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@@
 		(color 0 0 0 0)
+	)
+	(no_connect
+		(at 156.21 64.77)
+	)
+	(no_connect
+		(at 125.73 77.47)
+	)
+	(no_connect
+		(at 125.73 85.09)
+	)
+	(no_connect
+		(at 156.21 82.55)
+	)
+	(no_connect
+		(at 125.73 59.69)
+	)
+	(no_connect
+		(at 125.73 62.23)
+	)
+	(no_connect
+		(at 156.21 74.93)
+	)
+	(no_connect
+		(at 125.73 82.55)
+	)
+	(no_connect
+		(at 125.73 72.39)
+	)
+	(no_connect
+		(at 156.21 80.01)
+	)
+	(no_connect
+		(at 125.73 57.15)
+	)
+	(no_connect
+		(at 156.21 77.47)
+	)
+	(no_connect
+		(at 156.21 57.15)
+	)
+	(no_connect
+		(at 125.73 69.85)
+	)
+	(no_connect
+		(at 156.21 62.23)
 	)
 	(wire
@@
 			)
 		)
-		(property "Footprint" "LED_THT:LED_D5.0mm_Horizontal_O1.27mm_Z15.0mm"
+		(property "Footprint" "LED_THT:LED_D5.0mm"
 			(at 191.77 81.28 0)
 			(effects
@@
 			)
 		)
-		(property "Footprint" "LED_THT:LED_D5.0mm_Horizontal_O1.27mm_Z15.0mm"
+		(property "Footprint" "LED_THT:LED_D5.0mm"
 			(at 191.77 58.42 0)
 			(effects
